Commit message: fix some imu gravity and tf, but lidar odometry still produce wrong odom

File: LIO-SAM/config/robot.urdf.xacro (robot description, xacro)
@@ -13,5 +13,5 @@
     <parent link="chassis_link" />
     <child link="imu_link_ned" />
-    <origin xyz="0 0 0" rpy="${PI} 0 0" />
+    <origin xyz="0 0 0" rpy="0 0 0" />
   </joint>
   <link name="rslidar"> </link>

Commit message: 0313

File: LIO-SAM/config/robot.urdf.xacro (robot description, xacro)
@@ -9,8 +9,8 @@
     <origin xyz="0 0 0" rpy="0 0 0" />
   </joint>
-  <link name="imu_link_ned"> </link>
+  <link name="imu_link"> </link>
   <joint name="imu_joint" type="fixed">
     <parent link="chassis_link" />
-    <child link="imu_link_ned" />
+    <child link="imu_link" />
     <origin xyz="0 0 0" rpy="0 0 0" />
   </joint>
@@ -19,5 +19,5 @@
     <parent link="chassis_link" />
     <child link="rslidar" />
-    <origin xyz="0.425 0.075 1.728" rpy="0 0 0" />
+    <origin xyz="0.0 0.0 0.0" rpy="0 0 0" />
   </joint>
   <link name="navsat_link"> </link>
